File: qazivan_m/qazivan_m.kicad_pcb (KiCad board)
At the start: 2 copper layers, 204.8 x 95.2 mm, 121 parts, among them J1 AVR-ISP-6, J3 Conn_01x04_Female, U1 ATmega32U4-AU, Y1 16MHz

Commit message: update bottom row
Parts:
- MX33: footprint MX_Only:MXOnly-1U-Hotswap -> MX_Only:MXOnly-2.25U-Hotswap-ReversedStabilizers
- MX34: footprint MX_Only:MXOnly-2.25U-Hotswap-ReversedStabilizers -> MX_Only:MXOnly-2U-Hotswap-ReversedStabilizers
- MX35: footprint MX_Only:MXOnly-2U-Hotswap-ReversedStabilizers -> MX_Only:MXOnly-1U-Hotswap
- MX38: footprint MX_Only:MXOnly-6.25U-Hotswap-ReversedStabilizers -> MX_Only:MXOnly-6.25U-Hotswap
- moved MX34 21.3 mm to (159.1, 118.7)
- moved D33 14.9 mm to (101.5, 109.0)
- moved MX33 11.9 mm to (118.6, 118.7)
- moved MX35 9.38 mm to (187.7, 118.7)
- moved D35 7.48 mm to (178.0, 109.0)
- moved D34 6.13 mm to (140.1, 109.0)
- turned MX38 to 180 degrees
Connections:
- MX34 pad 1: COL4 -> COL5
- MX35 pad 1: COL5 -> COL7
- MX36 pad 1: COL7 -> COL8
- MX38 pad 2: Net-(D35-Pad2) -> Net-(D34-Pad2)
Routing:
- net Net-(D34-Pad2): track 4.94 -> 47.7 mm, vias 0 -> 1
- net Net-(D33-Pad2): track 6.22 -> 28.9 mm
- net COL4: track 150.7 -> 129.8 mm, vias 6 -> 5
- net COL8: track 181.3 -> 201.5 mm, vias 3 -> 4
- net COL7: track 194.5 -> 182.8 mm
- net COL5: track 200.5 -> 191.6 mm
- net Net-(D35-Pad2): track 26.2 -> 18.1 mm
- net COL3: track 150.4 -> 149.0 mm
- net GND: vias 32 -> 33
Other:
- board text added: "2.25u"
- board text added: "2.25u 6.25u"
- board text added: "2u"
- board text added: "6.25u"
