File: qazivan_m/qazivan_m.kicad_pcb (KiCad board)
At the start: 2 copper layers, 204.8 x 95.2 mm, 121 parts, among them J1 AVR-ISP-6, J3 Conn_01x04_Female, U1 ATmega32U4-AU, Y1 16MHz

Commit message: center big bar
Parts:
- MX45: renamed from MX38; footprint MX_Only:MXOnly-6.25U-Hotswap -> MX_Only:MXOnly-6.25U-Hotswap-ReversedStabilizers
- moved MX45 18.9 mm to (137.8, 118.7), turned to 0 degrees
- moved D44 11.4 mm to (151.5, 109.0)
- renumbered D46 to D1, D1 to D10, D2 to D11, D3 to D12, D4 to D13, D5 to D14, D6 to D15, D7 to D16, D8 to D17, D9 to D18, D10 to D19, D40 to D2, D11 to D20, D12 to D21, D13 to D22, D14 to D23, D15 to D24, D16 to D25, D17 to D26, D18 to D27, D19 to D28, D20 to D29, D41 to D3, D21 to D30, D22 to D31, D23 to D32, D24 to D33, D25 to D34, D26 to D35, D27 to D36, D28 to D37, D39 to D38, D29 to D39, D42 to D4, D30 to D40, D31 to D41, D32 to D42, D33 to D43, D34 to D44, D35 to D45, D36 to D46, D37 to D47, D38 to D48, D43 to D5, D44 to D6, D45 to D7, D47 to D8, D48 to D9, J3 to J1, J1 to J2, MX40 to MX1, MX4 to MX10, MX5 to MX11, MX6 to MX12, MX7 to MX13, MX8 to MX14, MX9 to MX15, MX10 to MX16, MX11 to MX17, MX12 to MX18, MX13 to MX19, MX41 to MX2, MX14 to MX20, MX15 to MX21, MX16 to MX22, MX17 to MX23, MX18 to MX24, MX19 to MX25, MX20 to MX26, MX21 to MX27, MX22 to MX28, MX23 to MX29, MX42 to MX3, MX24 to MX30, MX25 to MX31, MX26 to MX32, MX27 to MX33, MX28 to MX34, MX39 to MX35, MX29 to MX36, MX30 to MX37, MX31 to MX38, MX32 to MX39, MX43 to MX4, MX33 to MX40, MX34 to MX41, MX35 to MX42, MX36 to MX43, MX37 to MX44, MX44 to MX5, MX45 to MX6, MX1 to MX7, MX2 to MX8, MX3 to MX9, R7 to R1, R8 to R2, R9 to R3, R1 to R4, R2 to R5, R3 to R6, R4 to R7, R5 to R8, R6 to R9
Routing:
- net ROW3: track 260.7 -> 234.1 mm
- net Net-(D44-Pad2): track 47.7 -> 26.0 mm, vias 1 -> 0
- net COL5: track 191.6 -> 195.1 mm, vias 6 -> 7
Other:
- board text removed: "2.25u 6.25u"
